Commit message: Updated urdf file for matching the new real robot

File: src/bringup/config/robot_description/diff_drive.urdf.xacro (robot description, xacro)
@@ -10,15 +10,19 @@
   </link>
   <link name="base_link">
+  </link>
+  <joint name="chassis_joint" type="fixed">
+    <parent link="base_link" />
+    <child link="chassis" />
+    <origin rpy="0 0 0" xyz="0 0 0" />
+  </joint>
+  <link name="chassis">
     <visual>
-      <origin xyz="0 0 0" rpy="0 0 0" />
+      <origin rpy="1.57 0 1.57" xyz="0 0 0" />
       <geometry>
-        <box size="0.21 0.2 0.11" />
+        <mesh filename="package://robot_description/urdf/meshes/AssiemeBaseLink.dae" />
       </geometry>
-      <material name="blue">
-        <color rgba="0 0.5 1 1" />
-      </material>
     </visual>
     <collision>
-      <origin xyz="0 0 0.068" rpy="0 0 0" />
+      <origin rpy="0 0 0" xyz="-0.03 0 0" />
       <geometry>
         <box size="0.21 0.2 0.11" />
@@ -26,5 +30,5 @@
     </collision>
     <inertial>
-      <mass value="5" />
+      <mass value="5.0" />
       <inertia ixx="0.13" ixy="0.0" ixz="0.0" iyy="0.21" iyz="0.0" izz="0.13" />
     </inertial>
@@ -32,7 +36,7 @@
   <link name="caster">
     <visual>
-      <origin xyz="0.0 0 0" rpy="0 0 0" />
+      <origin xyz="0 0 0" rpy="1.57 0 0" />
       <geometry>
-        <sphere radius="0.033" />
+        <mesh filename="package://robot_description/urdf/meshes/caster.dae" />
       </geometry>
       <material name="darkgray">
@@ -58,11 +62,8 @@
   <link name="right_wheel">
     <visual>
-      <origin xyz="0 0 0" rpy="1.570795 0 0" />
+      <origin xyz="0 0.015 0" rpy="0 0 0" />
       <geometry>
-        <cylinder length="0.026" radius="0.033" />
+        <mesh filename="package://robot_description/urdf/meshes/wheel.dae" />
       </geometry>
-      <material name="darkgray">
-        <color rgba=".2 .2 .2 1" />
-      </material>
     </visual>
     <collision>
@@ -80,16 +81,13 @@
     <parent link="base_link" />
     <child link="right_wheel" />
-    <origin xyz="-0.09 -0.1 -0.035" rpy="0 0 0" />
+    <origin xyz="-0.12 -0.11 -0.059" rpy="0 0 0" />
     <axis xyz="0 1 0" />
   </joint>
   <link name="left_wheel">
     <visual>
-      <origin xyz="0 0 0" rpy="1.570795 0 0" />
+      <origin xyz="0 -0.015 0" rpy="0 0 3.14" />
       <geometry>
-        <cylinder length="0.026" radius="0.033" />
+        <mesh filename="package://robot_description/urdf/meshes/wheel.dae" />
       </geometry>
-      <material name="darkgray">
-        <color rgba=".2 .2 .2 1" />
-      </material>
     </visual>
     <collision>
@@ -107,5 +105,5 @@
     <parent link="base_link" />
     <child link="left_wheel" />
-    <origin xyz="-0.09 0.1 -0.035" rpy="0 0 0" />
+    <origin xyz="-0.12 0.11 -0.059" rpy="0 0 0" />
     <axis xyz="0 1 0" />
   </joint>
@@ -113,18 +111,17 @@
     <parent link="base_link" />
     <child link="laser" />
-    <origin xyz="0 0 0.055" rpy="0 0 0" />
+    <origin xyz="-0.035 0 0.1" rpy="0 0 0" />
   </joint>
   <link name="laser">
     <visual>
+      <origin xyz="0 0 0" rpy="1.57 0 0" />
       <geometry>
-        <cylinder radius="0.05" length="0.06" />
+        <mesh filename="package://robot_description/urdf/meshes/rp_lidar_a1.dae" />
       </geometry>
-      <material name="darkgray">
-        <color rgba=".2 .2 .2 1" />
-      </material>
     </visual>
     <collision>
+      <origin xyz="0 0 -0.03" rpy="0 0 0" />
       <geometry>
-        <cylinder radius="0.05" length="0.06" />
+        <cylinder radius="0.05" length="0.04" />
       </geometry>
     </collision>
@@ -137,15 +134,12 @@
     <parent link="base_link" />
     <child link="imu" />
-    <origin xyz="-0.105 0 0" rpy="0 0 0" />
+    <origin xyz="-0.123 0 0.005" rpy="0 0 0" />
   </joint>
   <link name="imu">
     <visual>
-      <origin xyz="0 0 0" rpy="0 0 0" />
+      <origin xyz="0 0 0" rpy="1.57 0 0" />
       <geometry>
-        <box size="0.026 0.02 0.002" />
+        <mesh filename="package://robot_description/urdf/meshes/Adafruit_BNO055_AP297.dae" />
       </geometry>
-      <material name="darkgray">
-        <color rgba=".2 .2 .2 1" />
-      </material>
     </visual>
     <collision>
@@ -161,5 +155,5 @@
   </link>
   <xacro:sensor_d435 parent="base_link" name="camera0" use_nominal_extrinsics="true">
-    <origin xyz="0.1 0.0 0.055" rpy="0 0 0" />
+    <origin xyz="0.070 0.0 0.055" rpy="0 0 0" />
   </xacro:sensor_d435>
   <ros2_control name="dd_robot_control" type="system">
